File: freedom MKL05Z/veiculo_MKL05Z/veiculo_MLK05Z.kicad_pcb (KiCad board)
At the start: 2 copper layers, 68.6 x 54.6 mm, 58 parts, among them J1 Conn_01x02_Male, J10 Conn_01x02_Male, J11 Conn_01x02_Male, J12 Conn_01x02_Male, J13 Conn_01x02_Male, J14 Conn_01x02_Male, J15 Conn_01x02_Male, J16 Conn_01x02_Male, J17 Conn_01x02_Male, J18 Conn_01x02_Male, J19 Conn_01x02_Male, J2 Conn_01x02_Male, J20 Conn_01x02_Male, J21 Conn_01x02_Male, J23 Conn_01x04_Male, J3 Conn_01x02_Male, J4 Conn_01x02_Male, J5 Conn_01x02_Male, J6 Conn_01x02_Male, J7 Conn_02x13_Odd_Even, J8 Conn_01x02_Male, J9 Conn_01x02_Male, P1 Power, P2 Analog, P3 Digital, P4 Digital, P6 CONN_01X01, P7 CONN_01X01, P8 CONN_01X01, Q1 2N7002, Q3 2N7002, Q4 2N7002, Q5 2N7002, Q6 2N7002, Q7 2N7002, Q8 2N7002, Q9 2N7002

Commit message: Created README.md to MKL05Z Shield
Connections:
- J19 pad 2: 11 -> 10
Routing:
- net 10: track 0.00 -> 4.14 mm
- net 11: track 4.09 -> 0.00 mm
- net GND: vias 3 -> 2
Changed lines of the file:
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@@
       (net 38 "PWM2") (pinfunction "Pin_1") (pintype "passive"))
     (pad "2" thru_hole roundrect (at 0 2.54 180) (size 1.7272 2.032) (drill 1.016) (layers "*.Cu" "*.Mask" "F.SilkS") (roundrect_rratio 0.25)
-      (net 15 "11") (pinfunction "Pin_2") (pintype "passive"))
+      (net 16 "10") (pinfunction "Pin_2") (pintype "passive"))
     (model "${KISYS3DMOD}/Connector_PinHeader_2.54mm.3dshapes/PinHeader_1x02_P2.54mm_Vertical.wrl"
       (offset (xyz 0 0 0))
@@
   (segment (start 149.098 119.253) (end 149.098 123.825) (width 0.508) (layer "B.Cu") (net 3))
   (segment (start 129.70764 94.45752) (end 132.24764 91.91752) (width 0.5) (layer "F.Cu") (net 4))
-  (segment (start 140.868 108.255) (end 140.868 95.725) (width 0.25) (layer "F.Cu") (net 4))
+  (segment (start 140.868 108.255) (end 140.868 95.725) (width 0.5) (layer "F.Cu") (net 4))
   (segment (start 140.868 95.725) (end 140.948 95.645) (width 0.25) (layer "F.Cu") (net 4))
   (segment (start 137.22052 91.91752) (end 140.948 95.645) (width 0.5) (layer "F.Cu") (net 4))
   (segment (start 132.24764 91.91752) (end 137.22052 91.91752) (width 0.5) (layer "F.Cu") (net 4))
   (via (at 175.768 99.695) (size 1.5) (drill 0.6) (layers "F.Cu" "B.Cu") (net 4))
-  (via (at 126.75 94.5) (size 1.5) (drill 0.6) (layers "F.Cu" "B.Cu") (free) (net 4))
   (via (at 112.4457 99.75) (size 1.5) (drill 0.6) (layers "F.Cu" "B.Cu") (net 4))
   (segment (start 151.638 123.825) (end 151.638 119.253) (width 0.508) (layer "B.Cu") (net 4))
@@
   (segment (start 144.825 91.025659) (end 144.825 91) (width 0.5) (layer "B.Cu") (net 14))
   (segment (start 145.7673 87.677661) (end 145.7673 84.168418) (width 0.25) (layer "B.Cu") (net 14))
-  (segment (start 145.034 75.565) (end 145.034 77.939) (width 0.508) (layer "B.Cu") (net 15))
-  (segment (start 145.034 77.939) (end 146.25 79.155) (width 0.508) (layer "B.Cu") (net 15))
+  (segment (start 146.25 79.155) (end 146.25 76.889) (width 0.508) (layer "B.Cu") (net 16))
+  (segment (start 146.25 76.889) (end 147.574 75.565) (width 0.508) (layer "B.Cu") (net 16))
   (segment (start 150.50625 88.575) (end 151.138711 88.575) (width 0.25) (layer "B.Cu") (net 18))
   (segment (start 149.5875 93.75) (end 149.5875 89.49375) (width 0.5) (layer "B.Cu") (net 18))
@@
   (segment (start 168.402 77.902) (end 166.878 76.378) (width 0.508) (layer "B.Cu") (net 23))
   (segment (start 166.878 76.378) (end 166.878 75.565) (width 0.508) (layer "B.Cu") (net 23))
-  (segment (start 172.25 77.25) (end 171.103 77.25) (width 0.25) (layer "B.Cu") (net 24))
+  (segment (start 173.5 86.319961) (end 173.5 78.07404) (width 0.25) (layer "B.Cu") (net 24))
   (segment (start 170.25 88.9375) (end 169.838618 88.9375) (width 0.25) (layer "B.Cu") (net 24))
-  (segment (start 173.5 86.319961) (end 173.5 78.5) (width 0.25) (layer "B.Cu") (net 24))
+  (segment (start 171.353 77.5) (end 169.418 75.565) (width 0.25) (layer "B.Cu") (net 24))
+  (segment (start 170.882461 88.9375) (end 173.5 86.319961) (width 0.25) (layer "B.Cu") (net 24))
   (segment (start 169.838618 88.9375) (end 167.776118 91) (width 0.25) (layer "B.Cu") (net 24))
-  (segment (start 170.882461 88.9375) (end 173.5 86.319961) (width 0.25) (layer "B.Cu") (net 24))
+  (segment (start 172.92596 77.5) (end 171.353 77.5) (width 0.25) (layer "B.Cu") (net 24))
+  (segment (start 170.25 88.9375) (end 170.882461 88.9375) (width 0.25) (layer "B.Cu") (net 24))
   (segment (start 167.776118 91) (end 167.625 91) (width 0.25) (layer "B.Cu") (net 24))
-  (segment (start 173.5 78.5) (end 172.25 77.25) (width 0.25) (layer "B.Cu") (net 24))
-  (segment (start 171.103 77.25) (end 169.418 75.565) (width 0.25) (layer "B.Cu") (net 24))
-  (segment (start 170.25 88.9375) (end 170.882461 88.9375) (width 0.25) (layer "B.Cu") (net 24))
+  (segment (start 173.5 78.07404) (end 172.92596 77.5) (width 0.25) (layer "B.Cu") (net 24))
   (segment (start 174.6872 88.342383) (end 173.6344 89.395183) (width 0.508) (layer "B.Cu") (net 25))
   (segment (start 173.6344 91.8656) (end 166 99.5) (width 0.508) (layer "B.Cu") (net 25))

Commit message: Update MKL05Z
Other:
- board text added: "Shield MKL05Z Equipe RoboRoadsters Adaptado de: Shield Arduino Uno Prof. Renan Augusto Starke"
- board text removed: "Shield MKL05Z Equipe RoboRoadsters Adapatado de: Shield Arduino Uno Prof. Renan Augusto Starke"
Changed lines of the file:
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@@
     (effects (font (size 1 1) (thickness 0.25)))
   )
-  (gr_text "Shield MKL05Z \nEquipe RoboRoadsters\n\nAdapatado de:\nShield Arduino Uno\nProf. Renan Augusto Starke" (at 150 101.75) (layer "F.SilkS")
+  (gr_text "Shield MKL05Z \nEquipe RoboRoadsters\n\nAdaptado de:\nShield Arduino Uno\nProf. Renan Augusto Starke" (at 150 101.75) (layer "F.SilkS")
     (effects (font (size 1 1) (thickness 0.1)))
   )

Commit message: CNC Files
Parts:
- moved J19 0.50 mm to (146.8, 81.7)
Routing:
- net L_TCRT: track 34.2 -> 35.5 mm
- net R_TCRT: track 32.4 -> 33.1 mm
